File: Binary_Display/Binary_Display.sch (KiCad schematic (older format))
At the start: 46 parts, among them U1 MAX_7219

Commit message: Changes
Parts:
- removed Conn1: Molex_SL_5, MRDT_Connectors:MOLEX_SL_5_Horizontal, symbol Molex_SL_5
- added J?: Conn_01x05, symbol Conn_01x05
Connections:
- net +5V: now also J?.1 (Pin_1)
- net Clk: now also J?.5 (Pin_5)
- net Din: now also J?.3 (Pin_3)
- net GND: now also J?.2 (Pin_2)
- net Load: now also J?.4 (Pin_4)
Changed lines of the file:
@@
 LIBS:MRDT_ICs
 LIBS:MRDT_Passives
+LIBS:MRDT_Sensors
 LIBS:MRDT_Shields
 LIBS:MRDT_Silkscreens
@@
 	1    3250 3700
 	1    0    0    -1
-$EndComp
-$Comp
-L Molex_SL_5 Conn1
-U 1 1 5B3D48C5
-P 1900 2550
-F 0 "Conn1" H 1950 2500 60  0001 C CNN
-F 1 "Molex_SL_5" H 1950 3100 60  0000 C CNN
-F 2 "MRDT_Connectors:MOLEX_SL_5_Horizontal" H 1900 2550 60  0001 C CNN
-F 3 "" H 1900 2550 60  0001 C CNN
-	1    1900 2550
-	-1   0    0    -1
 $EndComp
 Text Label 2850 3300 0    60   ~ 0
@@
 Wire Notes Line
 	7900 2700 7900 1000
+$Comp
+L Conn_01x05 J?
+U 1 1 5B6CA5A9
+P 1900 2300
+F 0 "J?" H 1900 2600 50  0000 C CNN
+F 1 "Conn_01x05" H 1900 2000 50  0000 C CNN
+F 2 "" H 1900 2300 50  0001 C CNN
+F 3 "" H 1900 2300 50  0001 C CNN
+	1    1900 2300
+	-1   0    0    -1
+$EndComp
 $EndSCHEMATC

Commit message: Made Clock Board
Parts:
- removed J?: Conn_01x05, symbol Conn_01x05
- added J1: ClockBoard, Project_Library:Clock_Board, symbol ClockBoard
Connections:
- net +5V: now also J1.VCC (Pin_1)
- net Clk: now also J1.CLK (Pin_5)
- net Din: now also J1.DIN (Pin_3)
- net GND: now also J1.GND (Pin_2)
- net Load: now also J1.CS (Pin_4)
Changed lines of the file:
@@
 	7900 2700 7900 1000
 $Comp
-L Conn_01x05 J?
-U 1 1 5B6CA5A9
+L ClockBoard J1
+U 1 1 5B744B1C
 P 1900 2300
-F 0 "J?" H 1900 2600 50  0000 C CNN
-F 1 "Conn_01x05" H 1900 2000 50  0000 C CNN
-F 2 "" H 1900 2300 50  0001 C CNN
+F 0 "J1" H 1900 2600 50  0000 C CNN
+F 1 "ClockBoard" H 1900 2000 50  0000 C CNN
+F 2 "Project_Library:Clock_Board" H 1900 2300 50  0001 C CNN
 F 3 "" H 1900 2300 50  0001 C CNN
 	1    1900 2300
