File: Binary_Display/Binary_Display.kicad_pcb (KiCad board)
At the start: 2 copper layers, 46 parts, among them U1 MAX_7219

Commit message: Changes
Parts:
- removed Conn1: Molex_SL_5, MRDT_Connectors:MOLEX_SL_5_Horizontal
- added J1: Conn_01x02, Socket_Strips:Socket_Strip_Straight_1x02_Pitch2.54mm, B.Cu at (191.0, 130.8)
- added J2: Conn_01x03, Socket_Strips:Socket_Strip_Straight_1x03_Pitch2.54mm, B.Cu at (201.5, 135.3)
- added REF**: 4_40_Hole, MRDT_Drill_Holes:4_40_Hole_Corner, F.Cu at (205.6, 81.9)
- added REF**: 4_40_Hole, MRDT_Drill_Holes:4_40_Hole_Corner, F.Cu at (124.7, 136.2)
- added REF**: 4_40_Hole, MRDT_Drill_Holes:4_40_Hole_Corner, F.Cu at (205.6, 136.2)
- added REF**: 4_40_Hole, MRDT_Drill_Holes:4_40_Hole_Corner, F.Cu at (124.7, 81.9)
Other:
- board outline added: 96.9 x 70.4 mm
- board text added: "Day"
- board text added: "Hour"
- board text added: "Minute"
- board text added: "Month"
- board text added: "Second"
- board text added: "Week"
- board text added: "Week Day"
- board text added: "Year"

Commit message: Made Clock Board
Parts:
- removed J2: Conn_01x03, Socket_Strips:Socket_Strip_Straight_1x03_Pitch2.54mm
- J1: value Conn_01x02 -> ClockBoard; footprint Socket_Strips:Socket_Strip_Straight_1x02_Pitch2.54mm -> Project_Library:Clock_Board; moved to F.Cu
- moved J1 4.56 mm to (193.1, 134.9), turned to 90 degrees
Routing:
- net /Clk: track 0.00 -> 54.8 mm, vias 0 -> 2
- net /Din: track 0.00 -> 53.7 mm, vias 0 -> 2
- net /Load: track 0.00 -> 42.9 mm, vias 0 -> 2
- net /GND: track 5.35 -> 12.0 mm
- net Sec: track 69.3 -> 68.6 mm
- added copper zone on F.Cu, net /+5V
- added copper zone on B.Cu, net /GND

Commit message: generated Gerbs
Changed lines of the file:
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@@
-(kicad_pcb (version 4) (host pcbnew 4.0.7)
+(kicad_pcb (version 20171130) (host pcbnew "(5.0.0)")
   (general
-    (links 94)
-    (no_connects 0)
-    (area 116.412599 73.638999 215.3978 144.547001)
     (thickness 1.6)
     (drawings 16)
@@
   )
   (setup
-    (last_trace_width 0.4064)
+    (last_trace_width 0.25)
     (user_trace_width 0.254)
     (user_trace_width 0.4064)
@@
     (visible_elements 7FFFFFFF)
     (pcbplotparams
-      (layerselection 0x00030_80000001)
+      (layerselection 0x010fc_ffffffff)
       (usegerberextensions false)
+      (usegerberattributes false)
+      (usegerberadvancedattributes false)
+      (creategerberjobfile false)
       (excludeedgelayer true)
       (linewidth 0.100000)
@@
       (hpglpennumber 1)
       (hpglpenspeed 20)
-      (hpglpendiameter 15)
-      (hpglpenoverlay 2)
+      (hpglpendiameter 15.000000)
       (psnegative false)
       (psa4output false)
@@
       (outputformat 1)
       (mirror false)
-      (drillshape 1)
+      (drillshape 0)
       (scaleselection 1)
-      (outputdirectory ""))
+      (outputdirectory "Gerbs/"))
   )
   (net 0 "")
@@
     (tags "SOIC 1.27")
     (attr smd)
-    (fp_text reference U1 (at 0 -8.8 270) (layer F.SilkS)
+    (fp_text reference U1 (at -3.176 -8.636 270) (layer F.SilkS)
       (effects (font (size 1 1) (thickness 0.15)))
     )
@@
     (tags "capacitor 0603")
     (attr smd)
-    (fp_text reference C1 (at 2.86 0 90) (layer F.SilkS)
+    (fp_text reference C1 (at -2.474 0 180) (layer F.SilkS)
       (effects (font (size 1 1) (thickness 0.15)))
     )
@@
     (tags "resistor 0603")
     (attr smd)
-    (fp_text reference R1 (at 2.964 0 90) (layer F.SilkS)
+    (fp_text reference R1 (at -2.624 0 180) (layer F.SilkS)
       (effects (font (size 1 1) (thickness 0.15)))
     )
@@
   (module Project_Library:Clock_Board (layer F.Cu)
     (at 193.0908 134.874 90)
-    (fp_text reference J1 (at 4.4704 -2.404201 90) (layer F.SilkS)
-      (effects (font (size 1 1) (thickness 0.15)))
-    )
+    (fp_text reference J1 (at 4.4704 -2.404201 90) (layer F.SilkS) hide
+      (effects (font (size 1 1) (thickness 0.15)))
+    )

Commit message: Added silkscreen to boards and organized gerbs
Parts:
- added G***: LOGO, MRDT_Silkscreens:z_sig_Andrew_Van_Horn_Sig_15mm, B.Cu at (172.7, 114.3)
Other:
- board text added: "+5V"
- board text added: "Binary Display, Rev 2 Andrew Van Horn"
- board text added: "Clk"
- board text added: "Din"
- board text added: "GND"
- board text added: "Load"
