File: Conventional_Display/Conventional_Display.sch (KiCad schematic (older format))
At the start: 93 parts, among them J1 Conn_01x05_Female, U1 7-Segment_Display_CA, U10 7-Segment_Display_CA, U11 7-Segment_Display_CA, U12 7-Segment_Display_CA, U13 7-Segment_Display_CA, U14 7-Segment_Display_CA, U15 7-Segment_Display_CA, U16 MAX_7219, U17 MAX_7219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

Commit message: Changes
Parts:
- removed J1: Conn_01x05_Female, MRDT_Connectors:MOLEX_SL_5_Horizontal, symbol Conn_01x05_Female
- added J?: Conn_01x05, symbol Conn_01x05
Connections:
- net +5V: now also J?.1 (Pin_1)
- net Clk: now also J?.5 (Pin_5)
- net Din: now also J?.3 (Pin_3)
- net GND: now also J?.2 (Pin_2)
- net Load: now also J?.4 (Pin_4)
Changed lines of the file:
@@
 $EndDescr
-$Comp
-L Conn_01x05_Female J1
-U 1 1 5B441E73
-P 4300 3750
-F 0 "J1" H 4250 3500 50  0000 C CNN
-F 1 "Conn_01x05_Female" H 4300 3450 50  0001 C CNN
-F 2 "MRDT_Connectors:MOLEX_SL_5_Horizontal" H 4300 3750 50  0001 C CNN
-F 3 "" H 4300 3750 50  0001 C CNN
-	1    4300 3750
-	-1   0    0    -1
-$EndComp
 $Comp
 L 1088A5_8x8_LED_Matrix U20
@@
 Conn
 Wire Notes Line
-	4250 4050 4800 4050
+	4200 4050 4800 4050
 Wire Notes Line
 	4800 4050 4800 3200
 Wire Notes Line
-	4800 3200 4250 3200
-Wire Notes Line
-	4250 3200 4250 4050
-Wire Notes Line
-	4250 3450 4800 3450
+	4800 3200 4200 3200
+Wire Notes Line
+	4200 3450 4800 3450
 Wire Wire Line
 	1700 5050 1700 5100
@@
 Wire Wire Line
 	5950 7650 5950 7700
+Wire Notes Line
+	4200 3200 4200 4050
+$Comp
+L Conn_01x05 J?
+U 1 1 5B6CA188
+P 4300 3750
+F 0 "J?" H 4300 4050 50  0000 C CNN
+F 1 "Conn_01x05" H 4300 3450 50  0000 C CNN
+F 2 "" H 4300 3750 50  0001 C CNN
+F 3 "" H 4300 3750 50  0001 C CNN
+	1    4300 3750
+	-1   0    0    -1
+$EndComp
 $EndSCHEMATC

Commit message: Made Clock Board
Parts:
- J1: renamed from J?; footprint (none) -> Project_Library:Clock_Board; symbol Conn_01x05 -> ClockBoard
Connections:
- net +5V: now also J1.VCC (Pin_1); no longer J1.1 (Pin_1)
- net Clk: now also J1.CLK (Pin_5); no longer J1.5 (Pin_5)
- net Din: now also J1.DIN (Pin_3); no longer J1.3 (Pin_3)
- net GND: now also J1.GND (Pin_2); no longer J1.2 (Pin_2)
- net Load: now also J1.CS (Pin_4); no longer J1.4 (Pin_4)
Changed lines of the file:
@@
 	4200 3200 4200 4050
 $Comp
-L Conn_01x05 J?
+L ClockBoard J1
 U 1 1 5B6CA188
 P 4300 3750
-F 0 "J?" H 4300 4050 50  0000 C CNN
+F 0 "J1" H 4300 4050 50  0000 C CNN
 F 1 "Conn_01x05" H 4300 3450 50  0000 C CNN
-F 2 "" H 4300 3750 50  0001 C CNN
+F 2 "Project_Library:Clock_Board" H 4300 3750 50  0001 C CNN
 F 3 "" H 4300 3750 50  0001 C CNN
 	1    4300 3750

Commit message: re routed conventional display LED matrix traces.
Parts:
- removed U20, U21, U22, U23: 1088A5_8x8_LED_Matrix, Project_Library:1088A5_8x8matrix, symbol 1088A5_8x8_LED_Matrix
- added U20, U21, U22, U23: 1088A5_8x8_LED_Matrix, Project_Library:1088A5_8x8matrix, symbol Project_Library:1088A5_8x8_LED_Matrix
- U16, U17, U18, U19: symbol MAX_7219 -> Project_Library:MAX_7219
Connections:
- net at U16.20 (Seg_C): now also U20.2 (Col_3)
- net at U16.3 (Dig_4): now also U20.9 (Row_4)
- net at U16.6 (Dig_2): now also U20.16 (Row_2)
- net at U16.23 (Seg_D): now also U20.14 (Col_4)
- net at U16.8 (Dig_7): now also U20.13 (Row_7)
- net at U16.16 (Seg_B): now also U20.12 (Col_2)
- net at U16.11 (Dig_1): now also U20.6 (Row_1)
- net at U16.2 (Dig_0): now also U20.1 (Row_0)
- net at U16.15 (Seg_F): now also U20.7 (Col_6)
- net at U16.7 (Dig_3): now also U20.4 (Row_3)
- net at U16.22 (Seg_DP): now also U20.5 (Col_0)
- net at U16.10 (Dig_5): now also U20.15 (Row_5)
- net at U16.5 (Dig_6): now also U20.10 (Row_6)
- net at U16.17 (Seg_G): now also U20.8 (Col_7)
- net at U16.21 (Seg_E): now also U20.3 (Col_5)
- net at U16.14 (Seg_A): now also U20.11 (Col_1)
- net at U17.20 (Seg_C): now also U21.2 (Col_3)
- net at U17.3 (Dig_4): now also U21.9 (Row_4)
- net at U17.6 (Dig_2): now also U21.16 (Row_2)
- net at U17.23 (Seg_D): now also U21.14 (Col_4)
- net at U17.8 (Dig_7): now also U21.13 (Row_7)
- net at U17.16 (Seg_B): now also U21.12 (Col_2)
- net at U17.11 (Dig_1): now also U21.6 (Row_1)
- net at U17.2 (Dig_0): now also U21.1 (Row_0)
- net at U17.15 (Seg_F): now also U21.7 (Col_6)
- net at U17.7 (Dig_3): now also U21.4 (Row_3)
- net at U17.22 (Seg_DP): now also U21.5 (Col_0)
- net at U17.10 (Dig_5): now also U21.15 (Row_5)
- net at U17.5 (Dig_6): now also U21.10 (Row_6)
- net at U17.17 (Seg_G): now also U21.8 (Col_7)
- net at U17.21 (Seg_E): now also U21.3 (Col_5)
- net at U17.14 (Seg_A): now also U21.11 (Col_1)
- net at U18.20 (Seg_C): now also U22.2 (Col_3)
- net at U18.3 (Dig_4): now also U22.9 (Row_4)
- net at U18.6 (Dig_2): now also U22.16 (Row_2)
- net at U18.23 (Seg_D): now also U22.14 (Col_4)
- net at U18.8 (Dig_7): now also U22.13 (Row_7)
- net at U18.16 (Seg_B): now also U22.12 (Col_2)
- net at U18.11 (Dig_1): now also U22.6 (Row_1)
- net at U18.2 (Dig_0): now also U22.1 (Row_0)
- net at U18.15 (Seg_F): now also U22.7 (Col_6)
- net at U18.7 (Dig_3): now also U22.4 (Row_3)
- net at U18.22 (Seg_DP): now also U22.5 (Col_0)
- net at U18.10 (Dig_5): now also U22.15 (Row_5)
- net at U18.5 (Dig_6): now also U22.10 (Row_6)
- net at U18.17 (Seg_G): now also U22.8 (Col_7)
- net at U18.21 (Seg_E): now also U22.3 (Col_5)
- net at U18.14 (Seg_A): now also U22.11 (Col_1)
- net at U19.20 (Seg_C): now also U23.2 (Col_3)
- net at U19.3 (Dig_4): now also U23.9 (Row_4)
- net at U19.6 (Dig_2): now also U23.16 (Row_2)
- net at U19.23 (Seg_D): now also U23.14 (Col_4)
- net at U19.8 (Dig_7): now also U23.13 (Row_7)
- net at U19.16 (Seg_B): now also U23.12 (Col_2)
- net at U19.11 (Dig_1): now also U23.6 (Row_1)
- net at U19.2 (Dig_0): now also U23.1 (Row_0)
- net at U19.15 (Seg_F): now also U23.7 (Col_6)
- net at U19.7 (Dig_3): now also U23.4 (Row_3)
- net at U19.22 (Seg_DP): now also U23.5 (Col_0)
- net at U19.10 (Dig_5): now also U23.15 (Row_5)
- net at U19.5 (Dig_6): now also U23.10 (Row_6)
- net at U19.17 (Seg_G): now also U23.8 (Col_7)
- net at U19.21 (Seg_E): now also U23.3 (Col_5)
- net at U19.14 (Seg_A): now also U23.11 (Col_1)
